Commit message: Update code

File: urdf/agv.urdf.xacro (robot description, xacro)
@@ -78,5 +78,5 @@
         <parent link="base_link"/>
         <child link="base_scan"/>
-        <origin xyz="-0.01 0.0 ${body_height}" rpy="0.0 0.0 0.0"/>
+        <origin xyz="-0.01 0.0 ${body_height + 0.09}" rpy="0.0 0.0 0.0"/>
     </joint>
     <!-- End Lidar -->
@@ -92,10 +92,10 @@
     <link name="uwb_link">
         <inertial>
-            <origin xyz="-0.01 0.024 -0.08" rpy="${PI/2} 0.0 0.0"/>
+            <origin xyz="0.0105 -0.024 -0.06" rpy="${PI/2} 0.0 ${PI}"/>
             <mass value="0.1" />
             <inertia ixx="0.001" ixy="0.0" ixz="0.0" iyy="0.001" iyz="0.0" izz="0.001" />
         </inertial>
         <visual>
-            <origin xyz="-0.01 0.024 -0.08" rpy="${PI/2} 0.0 0.0"/>
+            <origin xyz="0.0105 -0.024 -0.06" rpy="${PI/2} 0.0 ${PI}"/>
             <geometry>
                 <mesh filename="package://agv/meshs/uwb.STL" scale="0.001 0.001 0.001"/>
@@ -104,5 +104,5 @@
         </visual>
         <collision>
-            <origin xyz="-0.01 0.024 -0.08" rpy="${PI/2} 0.0 0.0"/>
+            <origin xyz="0.0105 -0.024 -0.06" rpy="${PI/2} 0.0 ${PI}"/>
             <geometry>
                 <mesh filename="package://agv/meshs/uwb.STL" scale="0.001 0.001 0.001"/>
@@ -113,5 +113,5 @@
         <parent link="base_link"/>
         <child link="uwb_link"/>
-        <origin xyz="-0.105 0.0 0.18" rpy="0.0 0.0 0.0"/>
+        <origin xyz="0.0 0.0 0.23" rpy="0.0 0.0 0.0"/>
     </joint>
     <!-- End UWB -->

Commit message: Change map

File: urdf/agv.urdf.xacro (robot description, xacro)
@@ -78,5 +78,5 @@
         <parent link="base_link"/>
         <child link="base_scan"/>
-        <origin xyz="-0.01 0.0 ${body_height + 0.09}" rpy="0.0 0.0 0.0"/>
+        <origin xyz="-0.03 0.0 ${body_height + 0.09}" rpy="0.0 0.0 0.0"/>
     </joint>
     <!-- End Lidar -->
@@ -113,5 +113,5 @@
         <parent link="base_link"/>
         <child link="uwb_link"/>
-        <origin xyz="0.0 0.0 0.23" rpy="0.0 0.0 0.0"/>
+        <origin xyz="-0.01 0.0 0.23" rpy="0.0 0.0 0.0"/>
     </joint>
     <!-- End UWB -->

Commit message: Backup code

File: urdf/agv.urdf.xacro (robot description, xacro)
@@ -78,5 +78,5 @@
         <parent link="base_link"/>
         <child link="base_scan"/>
-        <origin xyz="-0.03 0.0 ${body_height + 0.09}" rpy="0.0 0.0 0.0"/>
+        <origin xyz="0.0 0.0 ${body_height}" rpy="0.0 0.0 ${PI}"/>
     </joint>
     <!-- End Lidar -->
@@ -92,10 +92,10 @@
     <link name="uwb_link">
         <inertial>
-            <origin xyz="0.0105 -0.024 -0.06" rpy="${PI/2} 0.0 ${PI}"/>
+            <origin xyz="0.0105 -0.024 -0.055" rpy="${PI/2} 0.0 ${PI}"/>
             <mass value="0.1" />
             <inertia ixx="0.001" ixy="0.0" ixz="0.0" iyy="0.001" iyz="0.0" izz="0.001" />
         </inertial>
         <visual>
-            <origin xyz="0.0105 -0.024 -0.06" rpy="${PI/2} 0.0 ${PI}"/>
+            <origin xyz="0.0105 -0.024 -0.055" rpy="${PI/2} 0.0 ${PI}"/>
             <geometry>
                 <mesh filename="package://agv/meshs/uwb.STL" scale="0.001 0.001 0.001"/>
@@ -104,14 +104,20 @@
         </visual>
         <collision>
-            <origin xyz="0.0105 -0.024 -0.06" rpy="${PI/2} 0.0 ${PI}"/>
+            <origin xyz="0.0105 -0.024 -0.055" rpy="${PI/2} 0.0 ${PI}"/>
             <geometry>
                 <mesh filename="package://agv/meshs/uwb.STL" scale="0.001 0.001 0.001"/>
             </geometry>
         </collision>
+        <visual>
+            <origin xyz="-0.0825 0.035 -0.11" rpy="${PI/2} 0.0 0.0"/>
+            <geometry>
+                <mesh filename="package://agv/meshs/pad_uwb.STL" scale="0.001 0.001 0.001"/>
+            </geometry>
+        </visual>
     </link>
     <joint name="uwb_tag_joint" type="fixed">
         <parent link="base_link"/>
         <child link="uwb_link"/>
-        <origin xyz="-0.01 0.0 0.23" rpy="0.0 0.0 0.0"/>
+        <origin xyz="0.0 0.0 0.28" rpy="0.0 0.0 0.0"/>
     </joint>
     <!-- End UWB -->
